File: pcb/longboi.kicad_pcb (KiCad board)
At the start: 4 copper layers, 358 x 40 mm, 280 parts, among them J1 Testpad, J10 Conn_01x04_Pin, J11 Conn_01x02_Pin, J12 Conn_01x02_Pin, J13 Conn_01x02_Pin, J14 Conn_01x02_Pin, J15 Conn_01x03_Pin, J16 Conn_01x03_Pin, J17 Conn_01x03_Pin, J18 Conn_01x03_Pin, J19 Conn_01x02_Pin, J2 Testpad, J20 MX3.0, J21 MX3.0, J23 JST-XH, J24 JST-XH, J25 JST-XH, J26 JST-XH, J27 JST-XH, J28 JST-XH, J29 JST-XH, J3 Testpad, J30 JST-XH, J31 JST-XH, J32 JST-XH, J33 JST-XH, J34 JST-XH, J35 JST-XH, J36 JST-XH, J37 JST-XH, J38 JST-XH, J39 Conn_01x02_Pin, J4 Testpad, J40 Conn_01x03_Pin, J41 Conn_01x02_Pin, J42 JST-ZH, J44 Conn_01x02_Pin, J5 Testpad, J50 Conn_01x02_Pin, J6 JST-ZH, J7 Conn_01x04_Pin, J8 Conn_01x04_Pin, J9 Conn_01x04_Pin, Q1 HY1904C2, Q2 IRLML0030, Q4 IRLML0030, SW1 SW_SPST, SW2 SW_SPST, U1 STM32H723VGTx, U10 DRV8837, U11 DRV8837, U12 74LVC1G126, U13 74LVC1G126, U14 74LVC1G126, U15 74LVC1G126, U16 SN65HVD231, U17 TPS2116DRL, U18 TPS56637RPAR, U19 ME6211C33M5, U2 SN74LVC245APW, U20 SMF05CT1G-ES, U21 74LVC1G126, U22 74LVC1G126, U23 SMF05CT1G-ES, U3 SN74LVC245APW, U4 TMC2209-LA, U5 TMC2209-LA, U6 TMC2209-LA, U7 TMC2209-LA, U8 DRV8837, U9 DRV8837, Y1 Crystal_GND24

Commit message: fixes #15
Parts:
- moved R20 0.60 mm to (343.8, 103.4)
- turned SW1 to 180 degrees
- turned SW2 to 180 degrees
Connections:
- SW1 pad 2: NRST -> GND
- SW1 pad 3: (no net) -> NRST
- SW1 pad 4: (no net) -> NRST
- SW2 pad 2: BOOT0 -> +3.3V
- SW2 pad 3: (no net) -> BOOT0
- SW2 pad 4: (no net) -> BOOT0
Routing:
- net NRST: track 19.9 -> 23.8 mm
- net BOOT0: track 26.1 -> 30.0 mm
- net +3.3V: track 134.4 -> 137.8 mm
- net GND: track 224.8 -> 223.2 mm
- added copper zone on In1.Cu, net Net-(J20-Pin_1)
- removed copper zone on In1.Cu, net /24V_CAN/CANH

Commit message: fixes #5
Connections:
- R48 pad 2: /Endstops/Switch 4/SW -> /Endstops/Switch 3/SW
- R52 pad 2: /Endstops/Switch 3/SW -> /Endstops/Switch 4/SW
- R88 pad 1: /Endstops/Switch 4/SW -> /Endstops/Switch 3/SW
- R90 pad 1: /Endstops/Switch 3/SW -> /Endstops/Switch 4/SW
- U3 pad 8: /Endstops/Switch 3/SW -> /Endstops/Switch 4/SW
- U3 pad 9: /Endstops/Switch 4/SW -> /Endstops/Switch 3/SW
Routing:
- net /Endstops/Switch 4/SW: track 31.3 -> 24.5 mm
- net /Endstops/Switch 3/SW: track 24.5 -> 31.3 mm
Changed lines of the file:
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@@
 		)
 		(property ki_fp_filters "Connector*:*_1x??_*")
-		(sheetname "/Endstops/Switch 3/")
+		(sheetname "/Endstops/Switch 4/")
 		(sheetfile "switch.kicad_sch")
 		(attr through_hole)
@@
 		)
 		(property ki_fp_filters "LED* LED_SMD:* LED_THT:*")
-		(sheetname "/Endstops/Switch 4/")
+		(sheetname "/Endstops/Switch 3/")
 		(sheetfile "switch.kicad_sch")
 		(attr smd)
@@
 		)
 		(property ki_fp_filters "Connector*:*_1x??_*")
-		(sheetname "/Endstops/Switch 4/")
+		(sheetname "/Endstops/Switch 3/")
 		(sheetfile "switch.kicad_sch")
 		(attr through_hole)
@@
 		)
 		(property ki_fp_filters "R_*")
-		(sheetname "/Endstops/Switch 3/")
+		(sheetname "/Endstops/Switch 4/")
 		(sheetfile "switch.kicad_sch")
 		(attr smd)
@@
 			(layers "F.Cu" "F.Mask" "F.Paste")
 			(roundrect_rratio 0.25)
-			(net 182 "/Endstops/Switch 3/SW")
+			(net 183 "/Endstops/Switch 4/SW")
 			(pintype "passive")
 		)
@@
 		)
 		(property ki_fp_filters "R_*")
-		(sheetname "/Endstops/Switch 3/")
+		(sheetname "/Endstops/Switch 4/")
 		(sheetfile "switch.kicad_sch")
 		(attr smd)
@@
 		)
 		(property ki_fp_filters "LED* LED_SMD:* LED_THT:*")
-		(sheetname "/Endstops/Switch 3/")
+		(sheetname "/Endstops/Switch 4/")
 		(sheetfile "switch.kicad_sch")
 		(attr smd)
@@
 		)
 		(property ki_fp_filters "C_*")
-		(sheetname "/Endstops/Switch 3/")
+		(sheetname "/Endstops/Switch 4/")
 		(sheetfile "switch.kicad_sch")
 		(attr smd)
@@
 		)
 		(property ki_fp_filters "R_*")
-		(sheetname "/Endstops/Switch 4/")
+		(sheetname "/Endstops/Switch 3/")
 		(sheetfile "switch.kicad_sch")
 		(attr smd)
@@
 			(layers "F.Cu" "F.Mask" "F.Paste")
 			(roundrect_rratio 0.25)
-			(net 182 "/Endstops/Switch 3/SW")
+			(net 183 "/Endstops/Switch 4/SW")
 			(pinfunction "A7")
 			(pintype "bidirectional")
@@
 			(layers "F.Cu" "F.Mask" "F.Paste")
 			(roundrect_rratio 0.25)
-			(net 183 "/Endstops/Switch 4/SW")
+			(net 182 "/Endstops/Switch 3/SW")
 			(pinfunction "A8")
 			(pintype "bidirectional")
@@
 		)
 		(property ki_fp_filters "C_*")
-		(sheetname "/Endstops/Switch 4/")
+		(sheetname "/Endstops/Switch 3/")
 		(sheetfile "switch.kicad_sch")
 		(attr smd)
@@
 		)
 		(property ki_fp_filters "R_*")
-		(sheetname "/Endstops/Switch 4/")
+		(sheetname "/Endstops/Switch 3/")
 		(sheetfile "switch.kicad_sch")
 		(attr smd)
@@
 			(layers "F.Cu" "F.Mask" "F.Paste")
 			(roundrect_rratio 0.25)
-			(net 183 "/Endstops/Switch 4/SW")
+			(net 182 "/Endstops/Switch 3/SW")
 			(pintype "passive")
 		)
@@
 		)
 		(property ki_fp_filters "R_*")
-		(sheetname "/Endstops/Switch 4/")
+		(sheetname "/Endstops/Switch 3/")
 		(sheetfile "switch.kicad_sch")
 		(attr smd)
@@
 			(layers "F.Cu" "F.Mask" "F.Paste")
 			(roundrect_rratio 0.25)
-			(net 183 "/Endstops/Switch 4/SW")
+			(net 182 "/Endstops/Switch 3/SW")
 			(pintype "passive")
 		)
@@
 		)
 		(property ki_fp_filters "R_*")
-		(sheetname "/Endstops/Switch 3/")
+		(sheetname "/Endstops/Switch 4/")
 		(sheetfile "switch.kicad_sch")
 		(attr smd)
@@
 			(layers "F.Cu" "F.Mask" "F.Paste")
 			(roundrect_rratio 0.25)
-			(net 182 "/Endstops/Switch 3/SW")
+			(net 183 "/Endstops/Switch 4/SW")
 			(pintype "passive")
 		)
@@
 	)
 	(segment
-		(start 160.512552 115.825)
-		(end 162.5375 115.825)
+		(start 151.8 119)
+		(end 152.6 118.2)
 		(width 0.2)
 		(layer "F.Cu")
@@
 	)
 	(segment
-		(start 151.473 126.6)
-		(end 151.473 118.864552)
+		(start 151.8 135.625)
+		(end 151.8 133.6)
 		(width 0.2)
 		(layer "F.Cu")
@@
 	)
 	(segment
-		(start 150.6 129.825)
-		(end 151.473 128.952)
+		(start 151.8 133.6)
+		(end 151.8 119)
 		(width 0.2)
 		(layer "F.Cu")
@@
 	)
 	(segment
-		(start 152.464552 117.873)
-		(end 158.464552 117.873)
+		(start 152.6 118.2)
+		(end 158.6 118.2)
 		(width 0.2)
 		(layer "F.Cu")
@@
 	)
 	(segment
-		(start 151.473 128.952)
-		(end 151.473 126.6)
+		(start 158.6 118.2)
+		(end 160.325 116.475)
 		(width 0.2)
 		(layer "F.Cu")
@@
 	)
 	(segment
-		(start 158.464552 117.873)
-		(end 160.512552 115.825)
+		(start 150.625 133.6)
+		(end 151.8 133.6)
 		(width 0.2)
 		(layer "F.Cu")
@@
 	)
 	(segment
-		(start 150.625 126.6)
-		(end 151.473 126.6)
+		(start 150.6 136.825)
+		(end 151.8 135.625)
 		(width 0.2)
 		(layer "F.Cu")
@@
 	)
 	(segment
-		(start 151.473 118.864552)
-		(end 152.464552 117.873)
+		(start 160.325 116.475)
+		(end 162.5375 116.475)
 		(width 0.2)
 		(layer "F.Cu")
@@
 	)
 	(segment
-		(start 151.8 119)
-		(end 152.6 118.2)
+		(start 160.512552 115.825)
+		(end 162.5375 115.825)
 		(width 0.2)
 		(layer "F.Cu")
@@
 	)
 	(segment
-		(start 151.8 135.625)
-		(end 151.8 133.6)
+		(start 151.473 126.6)
+		(end 151.473 118.864552)
 		(width 0.2)
 		(layer "F.Cu")
@@
 	)
 	(segment
-		(start 151.8 133.6)
-		(end 151.8 119)
+		(start 150.6 129.825)
+		(end 151.473 128.952)
 		(width 0.2)
 		(layer "F.Cu")
@@
 	)
 	(segment
-		(start 152.6 118.2)
-		(end 158.6 118.2)
+		(start 152.464552 117.873)
+		(end 158.464552 117.873)
 		(width 0.2)
 		(layer "F.Cu")
@@
 	)
 	(segment
-		(start 158.6 118.2)
-		(end 160.325 116.475)
+		(start 151.473 128.952)
+		(end 151.473 126.6)
 		(width 0.2)
 		(layer "F.Cu")
@@
 	)
 	(segment
-		(start 150.625 133.6)
-		(end 151.8 133.6)
+		(start 158.464552 117.873)
+		(end 160.512552 115.825)
 		(width 0.2)
 		(layer "F.Cu")
@@
 	)
 	(segment
-		(start 150.6 136.825)
-		(end 151.8 135.625)
+		(start 150.625 126.6)
+		(end 151.473 126.6)
 		(width 0.2)
 		(layer "F.Cu")
@@
 	)
 	(segment
-		(start 160.325 116.475)
-		(end 162.5375 116.475)
+		(start 151.473 118.864552)
+		(end 152.464552 117.873)
 		(width 0.2)
 		(layer "F.Cu")

Commit message: fixes #10
Parts:
- added R26: 10k, Resistor_SMD:R_0603_1608Metric, F.Cu at (87.8, 113.6)
- added R27: 10k, Resistor_SMD:R_0603_1608Metric, F.Cu at (154.0, 112.0)
- added R67: 10k, Resistor_SMD:R_0603_1608Metric, F.Cu at (271.4, 114.2)
- added R68: 10k, Resistor_SMD:R_0603_1608Metric, F.Cu at (329.0, 109.8)
Routing:
- net GND: track 223.2 -> 234.0 mm
- net +3.3V: track 137.8 -> 139.7 mm
- net MOT3_SLP: track 51.8 -> 52.7 mm
- net MOT1_SLP: track 145.6 -> 146.3 mm
