File: pcb/longboi.kicad_pcb (KiCad board)
At the start: 4 copper layers, 358 x 40 mm, 284 parts, among them J1 Testpad, J10 Conn_01x04_Pin, J11 Conn_01x02_Pin, J12 Conn_01x02_Pin, J13 Conn_01x02_Pin, J14 Conn_01x02_Pin, J15 Conn_01x03_Pin, J16 Conn_01x03_Pin, J17 Conn_01x03_Pin, J18 Conn_01x03_Pin, J19 Conn_01x02_Pin, J2 Testpad, J20 MX3.0, J21 MX3.0, J23 JST-XH, J24 JST-XH, J25 JST-XH, J26 JST-XH, J27 JST-XH, J28 JST-XH, J29 JST-XH, J3 Testpad, J30 JST-XH, J31 JST-XH, J32 JST-XH, J33 JST-XH, J34 JST-XH, J35 JST-XH, J36 JST-XH, J37 JST-XH, J38 JST-XH, J39 Conn_01x02_Pin, J4 Testpad, J40 Conn_01x03_Pin, J41 Conn_01x02_Pin, J42 JST-ZH, J44 Conn_01x02_Pin, J5 Testpad, J50 Conn_01x02_Pin, J6 JST-ZH, J7 Conn_01x04_Pin, J8 Conn_01x04_Pin, J9 Conn_01x04_Pin, Q1 HY1904C2, Q2 IRLML0030, Q4 IRLML0030, SW1 SW_SPST, SW2 SW_SPST, U1 STM32H723VGTx, U10 DRV8837, U11 DRV8837, U12 74LVC1G126, U13 74LVC1G126, U14 74LVC1G126, U15 74LVC1G126, U16 SN65HVD231, U17 TPS2116DRL, U18 TPS56637RPAR, U19 ME6211C33M5, U2 SN74LVC245APW, U20 SMF05CT1G-ES, U21 74LVC1G126, U22 74LVC1G126, U23 SMF05CT1G-ES, U3 SN74LVC245APW, U4 TMC2209-LA, U5 TMC2209-LA, U6 TMC2209-LA, U7 TMC2209-LA, U8 DRV8837, U9 DRV8837, Y1 Crystal_GND24

Commit message: fixes #12
Parts:
- added RN1: 10k, Resistor_SMD:R_Array_Convex_4x0603, F.Cu at (252.8, 115.6)
- added RN2: 10k, Resistor_SMD:R_Array_Convex_4x0603, F.Cu at (256.1, 112.8)
- added RN3: 10k, Resistor_SMD:R_Array_Convex_4x0603, F.Cu at (175.3, 112.4)
- added RN4: 10k, Resistor_SMD:R_Array_Convex_4x0603, F.Cu at (171.7, 115.8)
- moved U2 5.60 mm to (262.4, 114.2)
- moved C14 5.38 mm to (256.8, 116.9)
Routing:
- net +3.3V: track 139.7 -> 159.1 mm, vias 38 -> 40
- net SW16: track 31.7 -> 37.9 mm, vias 0 -> 2
- net SW14: track 31.8 -> 38.0 mm, vias 0 -> 2
- net SW15: track 31.8 -> 37.9 mm, vias 0 -> 2
- net SW13: track 31.9 -> 38.0 mm
- net SW8: track 31.6 -> 37.6 mm, vias 0 -> 2
- net SW7: track 31.6 -> 37.2 mm, vias 0 -> 2
- net SW6: track 31.4 -> 37.0 mm, vias 0 -> 2
- net SW5: track 31.5 -> 37.1 mm, vias 0 -> 2
- net /Endstops/Switch 15/SW: track 121.4 -> 115.8 mm
- net /Endstops/Switch 13/SW: track 115.8 -> 110.2 mm
- net /Endstops/Switch 8/SW: track 99.0 -> 93.4 mm
- net /Endstops/Switch 7/SW: track 93.9 -> 88.3 mm
- net /Endstops/Switch 6/SW: track 30.5 -> 24.9 mm
- net /Endstops/Switch 5/SW: track 23.7 -> 18.1 mm
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Other:
- board text added: "Info"
- board text removed: "Katapult"
