File: pcb/24v_can.kicad_sch (KiCad schematic)
At the start: 7 parts, among them J19 Conn_01x02_Pin, J20 MX3.0, J21 MX3.0, U16 SN65HVD231

Commit message: fixes #9 fixes #4 fixes #13
Parts:
- added U23: SMF05CT1G-ES, Package_TO_SOT_SMD:SOT-363_SC-70-6, symbol LCSC:SMF05CT1G-ES
- F1: footprint Fuse:Fuseholder_Littelfuse_Nano2_157x -> Fuse:Fuseholder_Littelfuse_Nano2_154x
Connections:
- net GND: now also J20.2 (Pin_2), J21.2 (Pin_2), U23.2 (GND); no longer J20.1 (Pin_1), J21.1 (Pin_1)
- net CANH: now reaches J20.3 (Pin_3), J21.3 (Pin_3)
- net CANH: now also J19.2 (Pin_2), U16.7 (CANH), U23.6 (IO5); no longer R12.1, U16.6 (CANL)
- net CANL: now reaches J20.4 (Pin_4), J21.4 (Pin_4)
- net CANL: now also R12.1, U16.6 (CANL), U23.5 (IO4); no longer J19.2 (Pin_2), U16.7 (CANH)
- new net: F1.1, J20.1 (Pin_1), J21.1 (Pin_1)
- no-connect marks 1 -> 4
Other:
- moved on the sheet: J21

Commit message: specified some values and colors added lcsc part ids for all components
Parts:
- C52: LCSC (none) -> C14663
- F1: LCSC (none) -> C108518
- J19: LCSC (none) -> C492401
- J20, J21: LCSC (none) -> C277721
- R12: LCSC (none) -> C22787
- U16: LCSC (none) -> C129257
- U23: LCSC (none) -> C5180312
Changed lines of the file:
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@@
+			)
+		)
+		(property "LCSC" "C5180312"
+			(at 45.72 82.55 0)
+			(effects
+				(font
+					(size 1.27 1.27)
+				)
+				(hide yes)
 			)
 		)
@@
 			)
 		)
+		(property "LCSC" "C108518"
+			(at 132.08 46.99 0)
+			(effects
+				(font
+					(size 1.27 1.27)
+				)
+				(hide yes)
+			)
+		)
 		(pin "1"
 		)
@@
 			)
 		)
+		(property "LCSC" "C129257"
+			(at 80.0118 41.91 0)
+			(effects
+				(font
+					(size 1.27 1.27)
+				)
+				(hide yes)
+			)
+		)
 		(pin "4"
 		)
@@
 			)
 		)
+		(property "LCSC" "C22787"
+			(at 92.71 62.23 0)
+			(effects
+				(font
+					(size 1.27 1.27)
+				)
+				(hide yes)
+			)
+		)
 		(pin "1"
 		)
@@
 			)
 		)
+		(property "LCSC" "C277721"
+			(at 109.22 33.02 0)
+			(effects
+				(font
+					(size 1.27 1.27)
+				)
+				(hide yes)
+			)
+		)
 		(pin "4"
 		)
@@
 			)
 		)
+		(property "LCSC" "C277721"
+			(at 109.22 48.26 0)
+			(effects
+				(font
+					(size 1.27 1.27)
+				)
+				(hide yes)
+			)
+		)
 		(pin "4"
 		)
@@
 			)
 		)
+		(property "LCSC" "C492401"
+			(at 110.49 67.31 0)
+			(effects
+				(font
+					(size 1.27 1.27)
+				)
+				(hide yes)
+			)
+		)
 		(pin "1"
 		)
@@
 			(effects
 				(font
+					(size 1.27 1.27)
+				)
+				(hide yes)
+			)
+		)
+		(property "LCSC" "C14663"
+			(at 140.97 77.4763 0)
+			(effects
+				(font
