File: pcb/hp.kicad_sch (KiCad schematic)
At the start: 6 parts, among them J39 Conn_01x02_Pin, Q1 HY1904C2

Commit message: fixes #8: changed led series resistor values
Parts:
- R61: value 1.5k -> 3.3k
Changed lines of the file:
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@@
 		(fields_autoplaced yes)
 		(property "Reference" "R61"
-			(at 82.55 76.2 0)
+			(at 82.55 76.1999 0)
 			(effects
 				(font
@@
 			)
 		)
-		(property "Value" "1.5k"
-			(at 82.55 78.74 0)
+		(property "Value" "3.3k"
+			(at 82.55 78.7399 0)
 			(effects
 				(font

Commit message: fixes #6
Parts:
- R63: value 100k -> 10k
Changed lines of the file:
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@@
 		(fields_autoplaced yes)
 		(property "Reference" "R63"
-			(at 93.98 66.04 0)
+			(at 93.98 66.0399 0)
 			(effects
 				(font
@@
 			)
 		)
-		(property "Value" "100k"
-			(at 93.98 68.58 0)
+		(property "Value" "10k"
+			(at 93.98 68.5799 0)
 			(effects
 				(font

Commit message: specified some values and colors added lcsc part ids for all components
Parts:
- D5: value LED -> Red; LCSC (none) -> C965799
- J39: LCSC (none) -> C293362
- Q1: LCSC (none) -> C358116
- R61: LCSC (none) -> C22978
- R62: LCSC (none) -> C105588
- R63: LCSC (none) -> C98220
Changed lines of the file:
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@@
+			)
+		)
+		(property "LCSC" "C22978"
+			(at 82.55 76.1999 0)
+			(effects
+				(font
+					(size 1.27 1.27)
+				)
+				(hide yes)
 			)
 		)
@@
 			)
 		)
+		(property "LCSC" "C98220"
+			(at 93.98 66.0399 0)
+			(effects
+				(font
+					(size 1.27 1.27)
+				)
+				(hide yes)
+			)
+		)
 		(pin "1"
 		)
@@
 		(property "LCSC Part" "C358116"
 			(at 102.87 80.01 0)
+			(effects
+				(font
+					(size 1.27 1.27)
+				)
+				(hide yes)
+			)
+		)
+		(property "LCSC" "C358116"
+			(at 114.3 60.96 0)
 			(effects
 				(font
@@
 			)
 		)
+		(property "LCSC" "C293362"
+			(at 111.125 39.37 0)
+			(effects
+				(font
+					(size 1.27 1.27)
+				)
+				(hide yes)
+			)
+		)
 		(pin "2"
 		)
@@
 		(fields_autoplaced yes)
 		(property "Reference" "D5"
-			(at 83.82 68.8975 90)
+			(at 83.82 68.8974 90)
 			(effects
 				(font
@@
 			)
 		)
-		(property "Value" "LED"
-			(at 83.82 71.4375 90)
+		(property "Value" "Red"
+			(at 83.82 71.4374 90)
 			(effects
 				(font
@@
 			)
 		)
+		(property "LCSC" "C965799"
+			(at 83.82 68.8974 0)
+			(effects
+				(font
+					(size 1.27 1.27)
+				)
+				(hide yes)
+			)
+		)
 		(pin "1"
 		)
@@
 			(effects
 				(font
+					(size 1.27 1.27)
+				)
+				(hide yes)
+			)
+		)
+		(property "LCSC" "C105588"
+			(at 85.09 57.15 0)
+			(effects
+				(font
