File: pcb/reset_boot.kicad_sch (KiCad schematic)
At the start: 4 parts, among them SW1 SW_SPST, SW2 SW_SPST

Commit message: fixes #15
Parts:
- SW1, SW2: symbol Switch:SW_SPST -> Switch:SW_MEC_5E
Connections:
- net +3.3V: now also SW2.2
- net BOOT: now also SW2.3 (K), SW2.4 (A); no longer SW2.2 (B)
- net GND: now also SW1.2
- net RST: now also SW1.3 (K), SW1.4 (A); no longer SW1.2 (B)
Changed lines of the file:
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@@
+	)
+	(junction
+		(at 48.26 35.56)
+		(diameter 0)
+		(color 0 0 0 0)
 	)
 	(junction
@@
 		(color 0 0 0 0)
 	)
+	(junction
+		(at 48.26 59.69)
+		(diameter 0)
+		(color 0 0 0 0)
+	)
+	(wire
+		(pts
+			(xy 48.26 59.69) (xy 48.26 55.88)
+		)
+		(stroke
+			(width 0)
+			(type default)
+		)
+	)
 	(wire
 		(pts
@@
 	(wire
 		(pts
+			(xy 60.96 59.69) (xy 63.5 59.69)
+		)
+		(stroke
+			(width 0)
+			(type default)
+		)
+	)
+	(wire
+		(pts
+			(xy 50.8 33.02) (xy 48.26 33.02)
+		)
+		(stroke
+			(width 0)
+			(type default)
+		)
+	)
+	(wire
+		(pts
+			(xy 63.5 59.69) (xy 63.5 62.23)
+		)
+		(stroke
+			(width 0)
+			(type default)
+		)
+	)
+	(wire
+		(pts
 			(xy 63.5 43.18) (xy 63.5 45.72)
 		)
@@
 	(wire
 		(pts
+			(xy 63.5 33.02) (xy 63.5 35.56)
+		)
+		(stroke
+			(width 0)
+			(type default)
+		)
+	)
+	(wire
+		(pts
+			(xy 48.26 35.56) (xy 50.8 35.56)
+		)
+		(stroke
+			(width 0)
+			(type default)
+		)
+	)
+	(wire
+		(pts
 			(xy 48.26 62.23) (xy 48.26 59.69)
 		)
@@
 	(wire
 		(pts
+			(xy 48.26 33.02) (xy 48.26 35.56)
+		)
+		(stroke
+			(width 0)
+			(type default)
+		)
+	)
+	(wire
+		(pts
 			(xy 60.96 35.56) (xy 63.5 35.56)
 		)
@@
 	(wire
 		(pts
+			(xy 60.96 33.02) (xy 63.5 33.02)
+		)
+		(stroke
+			(width 0)
+			(type default)
+		)
+	)
+	(wire
+		(pts
+			(xy 48.26 59.69) (xy 50.8 59.69)
+		)
+		(stroke
+			(width 0)
+			(type default)
+		)
+	)
+	(wire
+		(pts
 			(xy 50.8 62.23) (xy 48.26 62.23)
-		)
-		(stroke
-			(width 0)
-			(type default)
-		)
-	)
-	(wire
-		(pts
-			(xy 48.26 35.56) (xy 50.8 35.56)
 		)
 		(stroke
@@
 	(symbol
 		(lib_id "power:+3.3V")
-		(at 48.26 59.69 0)
+		(at 48.26 55.88 0)
 		(unit 1)
 		(exclude_from_sim no)
@@
 		(fields_autoplaced yes)
 		(property "Reference" "#PWR0144"
-			(at 48.26 63.5 0)
+			(at 48.26 59.69 0)
 			(effects
 				(font
@@
 		)
 		(property "Value" "+3.3V"
-			(at 48.26 54.61 0)
+			(at 48.26 50.8 0)
 			(effects
 				(font
@@
 		)
 		(property "Footprint" ""
-			(at 48.26 59.69 0)
+			(at 48.26 55.88 0)
 			(effects
 				(font
@@
 		)
 		(property "Datasheet" ""
-			(at 48.26 59.69 0)
+			(at 48.26 55.88 0)
 			(effects
 				(font
@@
 		)
 		(property "Description" "Power symbol creates a global label with name \"+3.3V\""
-			(at 48.26 59.69 0)
+			(at 48.26 55.88 0)
 			(effects
 				(font
@@
 	)
 	(symbol
-		(lib_id "Switch:SW_SPST")
+		(lib_id "Switch:SW_MEC_5E")
 		(at 55.88 35.56 0)
 		(unit 1)
@@
 		(fields_autoplaced yes)
 		(property "Reference" "SW1"
-			(at 55.88 29.21 0)
+			(at 55.88 25.4 0)
 			(effects
 				(font
@@
 		)
 		(property "Value" "SW_SPST"
-			(at 55.88 31.75 0)
+			(at 55.88 27.94 0)
 			(effects
 				(font
@@
 		)
 		(property "Footprint" "LCSC:SW-SMD_4P-L3.4-W3.4-P2.00-LS4.0_TS3315A160GF"
+			(at 55.88 27.94 0)
+			(effects
+				(font
+					(size 1.27 1.27)
+				)
+				(hide yes)
+			)
+		)
+		(property "Datasheet" "http://www.apem.com/int/index.php?controller=attachment&id_attachment=1371"
+			(at 55.88 27.94 0)
+			(effects
+				(font
+					(size 1.27 1.27)
+				)
+				(hide yes)
+			)
+		)
+		(property "Description" "MEC 5E single pole normally-open tactile switch"
 			(at 55.88 35.56 0)
 			(effects
@@
 			)
 		)
-		(property "Datasheet" "~"
-			(at 55.88 35.56 0)
-			(effects
-				(font
-					(size 1.27 1.27)
-				)
-				(hide yes)
-			)
-		)
-		(property "Description" "Single Pole Single Throw (SPST) switch"
-			(at 55.88 35.56 0)
-			(effects
-				(font
-					(size 1.27 1.27)
-				)
-				(hide yes)
-			)
-		)
 		(pin "2"
 		)
 		(pin "1"
+		)
+		(pin "4"
+		)
+		(pin "3"
 		)
 		(instances
@@
 	)
 	(symbol
-		(lib_id "Switch:SW_SPST")
+		(lib_id "Switch:SW_MEC_5E")
 		(at 55.88 62.23 0)
 		(unit 1)
@@
 		(fields_autoplaced yes)
 		(property "Reference" "SW2"
-			(at 55.88 55.88 0)
+			(at 55.88 52.07 0)
 			(effects
 				(font
@@
 		)
 		(property "Value" "SW_SPST"
-			(at 55.88 58.42 0)
+			(at 55.88 54.61 0)
 			(effects
 				(font
@@
 		)
 		(property "Footprint" "LCSC:SW-SMD_4P-L3.4-W3.4-P2.00-LS4.0_TS3315A160GF"
+			(at 55.88 54.61 0)
+			(effects
+				(font
+					(size 1.27 1.27)
+				)
+				(hide yes)
+			)
+		)
+		(property "Datasheet" "http://www.apem.com/int/index.php?controller=attachment&id_attachment=1371"
+			(at 55.88 54.61 0)
+			(effects
+				(font
+					(size 1.27 1.27)
+				)
+				(hide yes)
+			)
+		)
+		(property "Description" "MEC 5E single pole normally-open tactile switch"
 			(at 55.88 62.23 0)
 			(effects
@@
 			)
 		)
-		(property "Datasheet" "~"
-			(at 55.88 62.23 0)
-			(effects
-				(font
-					(size 1.27 1.27)
-				)
-				(hide yes)
-			)
-		)
-		(property "Description" "Single Pole Single Throw (SPST) switch"
-			(at 55.88 62.23 0)
-			(effects
-				(font
-					(size 1.27 1.27)
-				)
-				(hide yes)
-			)
-		)
 		(pin "2"
 		)
 		(pin "1"
 		)
+		(pin "4"
+		)
+		(pin "3"
+		)
 		(instances

Commit message: specified some values and colors added lcsc part ids for all components
Parts:
- C62: LCSC (none) -> C14663
- R28: LCSC (none) -> C14675
- SW1, SW2: LCSC (none) -> C557593
Changed lines of the file:
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@@
+			)
+		)
+		(property "LCSC" "C14663"
+			(at 66.04 39.3763 0)
+			(effects
+				(font
+					(size 1.27 1.27)
+				)
+				(hide yes)
 			)
 		)
@@
 			)
 		)
+		(property "LCSC" "C14675"
+			(at 66.04 66.04 0)
+			(effects
+				(font
+					(size 1.27 1.27)
+				)
+				(hide yes)
+			)
+		)
 		(pin "1"
 		)
@@
 			)
 		)
+		(property "LCSC" "C557593"
+			(at 55.88 25.4 0)
+			(effects
+				(font
+					(size 1.27 1.27)
+				)
+				(hide yes)
+			)
+		)
 		(pin "2"
 		)
@@
 			(effects
 				(font
+					(size 1.27 1.27)
+				)
+				(hide yes)
+			)
+		)
+		(property "LCSC" "C557593"
+			(at 55.88 52.07 0)
+			(effects
+				(font
