File: pcb/rgb.kicad_sch (KiCad schematic)
At the start: 3 parts, among them J15 Conn_01x03_Pin, U12 74LVC1G126

Commit message: specified some values and colors added lcsc part ids for all components
Parts:
- C48: LCSC (none) -> C14663
- J15: LCSC (none) -> C565985
- U12: LCSC (none) -> C7394032
Changed lines of the file:
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@@
+			)
+		)
+		(property "LCSC" "C7394032"
+			(at 106.68 51.4061 0)
+			(effects
+				(font
+					(size 1.27 1.27)
+				)
+				(hide yes)
 			)
 		)
@@
 			)
 		)
+		(property "LCSC" "C14663"
+			(at 69.85 83.8136 0)
+			(effects
+				(font
+					(size 1.27 1.27)
+				)
+				(hide yes)
+			)
+		)
 		(pin "2"
 		)
@@
 			(effects
 				(font
+					(size 1.27 1.27)
+				)
+				(hide yes)
+			)
+		)
+		(property "LCSC" "C565985"
+			(at 124.46 57.15 0)
+			(effects
+				(font
