File: pcb/thermistor.kicad_sch (KiCad schematic)
At the start: 6 parts, among them J50 Conn_01x02_Pin

Commit message: specified some values and colors added lcsc part ids for all components
Parts:
- C82: LCSC (none) -> C14663
- D32: LCSC (none) -> C2500
- J50: LCSC (none) -> C378939
- R108, R109: LCSC (none) -> C705759
- R110: LCSC (none) -> C99782
Changed lines of the file:
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@@
+			)
+		)
+		(property "LCSC" "C378939"
+			(at 40.64 44.45 0)
+			(effects
+				(font
+					(size 1.27 1.27)
+				)
+				(hide yes)
 			)
 		)
@@
 			)
 		)
+		(property "LCSC" "C99782"
+			(at 52.07 38.1 0)
+			(effects
+				(font
+					(size 1.27 1.27)
+				)
+				(hide yes)
+			)
+		)
 		(pin "2"
 		)
@@
 			)
 		)
+		(property "LCSC" "C14663"
+			(at 88.9 48.2536 0)
+			(effects
+				(font
+					(size 1.27 1.27)
+				)
+				(hide yes)
+			)
+		)
 		(pin "2"
 		)
@@
 			)
 		)
+		(property "LCSC" "C705759"
+			(at 59.69 39.37 0)
+			(effects
+				(font
+					(size 1.27 1.27)
+				)
+				(hide yes)
+			)
+		)
 		(pin "2"
 		)
@@
 		(property "Description" "Resistor, small symbol"
 			(at 81.28 44.45 0)
+			(effects
+				(font
+					(size 1.27 1.27)
+				)
+				(hide yes)
+			)
+		)
+		(property "LCSC" "C705759"
+			(at 81.28 39.37 0)
 			(effects
 				(font
@@
 			(effects
 				(font
+					(size 1.27 1.27)
+				)
+				(hide yes)
+			)
+		)
+		(property "LCSC" "C2500"
+			(at 72.39 43.18 0)
+			(effects
+				(font
