File: pcb/steppers.kicad_sch (KiCad schematic)
At the start: 13 parts, among them J7 Conn_01x04_Pin, U4 TMC2209-LA

Commit message: specified some values and colors added lcsc part ids for all components
Parts:
- C16: LCSC (none) -> C21122
- C17: LCSC (none) -> C14663
- C18: LCSC (none) -> C23630
- C19: LCSC (none) -> C15849
- C20, C21: LCSC (none) -> C90142
- J7: LCSC (none) -> C566013
- R103, R95, R99: LCSC (none) -> C14675
- R4, R5: LCSC (none) -> C2934288
- U4: LCSC (none) -> C2150710
Changed lines of the file:
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@@
+			)
+		)
+		(property "LCSC" "C90142"
+			(at 161.29 59.6836 0)
+			(effects
+				(font
+					(size 1.27 1.27)
+				)
+				(hide yes)
 			)
 		)
@@
 		(property "Description" "Unpolarized capacitor, small symbol"
 			(at 149.86 60.96 0)
+			(effects
+				(font
+					(size 1.27 1.27)
+				)
+				(hide yes)
+			)
+		)
+		(property "LCSC" "C90142"
+			(at 152.4 59.6836 0)
 			(effects
 				(font
@@
 			)
 		)
+		(property "LCSC" "C23630"
+			(at 121.92 57.1436 0)
+			(effects
+				(font
+					(size 1.27 1.27)
+				)
+				(hide yes)
+			)
+		)
 		(pin "2"
 		)
@@
 			)
 		)
+		(property "LCSC" "C15849"
+			(at 139.7 59.6836 0)
+			(effects
+				(font
+					(size 1.27 1.27)
+				)
+				(hide yes)
+			)
+		)
 		(pin "2"
 		)
@@
 			)
 		)
+		(property "LCSC" "C14675"
+			(at 59.69 63.5 0)
+			(effects
+				(font
+					(size 1.27 1.27)
+				)
+				(hide yes)
+			)
+		)
 		(pin "1"
 		)
@@
 			)
 		)
+		(property "LCSC" "C2150710"
+			(at 89.154 88.392 0)
+			(effects
+				(font
+					(size 1.27 1.27)
+				)
+				(hide yes)
+			)
+		)
 		(pin "29"
 		)
@@
 			)
 		)
+		(property "LCSC" "C566013"
+			(at 130.81 40.64 0)
+			(effects
+				(font
+					(size 1.27 1.27)
+				)
+				(hide yes)
+			)
+		)
 		(pin "1"
 		)
@@
 			)
 		)
+		(property "LCSC" "C14675"
+			(at 46.99 46.99 0)
+			(effects
+				(font
+					(size 1.27 1.27)
+				)
+				(hide yes)
+			)
+		)
 		(pin "1"
 		)
@@
 			)
 		)
+		(property "LCSC" "C14675"
+			(at 77.47 86.36 0)
+			(effects
+				(font
+					(size 1.27 1.27)
+				)
+				(hide yes)
+			)
+		)
 		(pin "1"
 		)
@@
 			)
 		)
+		(property "LCSC" "C14663"
+			(at 86.36 27.9336 0)
+			(effects
+				(font
+					(size 1.27 1.27)
+				)
+				(hide yes)
+			)
+		)
 		(pin "2"
 		)
@@
 			)
 		)
+		(property "LCSC" "C2934288"
+			(at 121.92 83.82 0)
+			(effects
+				(font
+					(size 1.27 1.27)
+				)
+				(hide yes)
+			)
+		)
 		(pin "1"
 		)
@@
 			)
 		)
+		(property "LCSC" "C21122"
+			(at 67.31 52.0636 0)
+			(effects
+				(font
+					(size 1.27 1.27)
+				)
+				(hide yes)
+			)
+		)
 		(pin "2"
 		)
@@
 			(effects
 				(font
+					(size 1.27 1.27)
+				)
+				(hide yes)
+			)
+		)
+		(property "LCSC" "C2934288"
+			(at 130.81 83.82 0)
+			(effects
+				(font

Commit message: fixes #20 fixes #22 fixes #19
Parts:
- C20, C21: LCSC C90142 -> C6120020
Changed lines of the file:
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@@
 			)
 		)
-		(property "LCSC" "C90142"
+		(property "LCSC" "C6120020"
 			(at 161.29 59.6836 0)
 			(effects
@@
 			)
 		)
-		(property "LCSC" "C90142"
+		(property "LCSC" "C6120020"
 			(at 152.4 59.6836 0)
 			(effects
