File: pcb/longboi.kicad_sch (KiCad schematic)
At the start: 32 parts, among them J1 Testpad, J2 Testpad, J3 Testpad, J4 Testpad, J5 Testpad, J6 JST-PH, U1 STM32H723VGTx, Y1 25MHz

Commit message: get ready for production fixes #24 fixes #25
Parts:
- J6: LCSC C157997 -> C5305780
