File: pcb/usb.kicad_sch (KiCad schematic)
At the start: 2 parts, among them J42 JST-ZH, U20 SMF05CT1G-ES

Commit message: specified some values and colors added lcsc part ids for all components
Parts:
- J42: LCSC (none) -> C157997
- U20: LCSC (none) -> C5180312
Changed lines of the file:
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@@
+			)
+		)
+		(property "LCSC" "C157997"
+			(at 29.845 55.88 0)
+			(effects
+				(font
+					(size 1.27 1.27)
+				)
+				(hide yes)
 			)
 		)
@@
 			(effects
 				(font
+					(size 1.27 1.27)
+				)
+				(hide yes)
+			)
+		)
+		(property "LCSC" "C5180312"
+			(at 144.78 52.07 0)
+			(effects
+				(font

Commit message: wip
Parts:
- removed J42: JST-ZH, Connector_JST:JST_ZH_B4B-ZR_1x04_P1.50mm_Vertical, symbol Connector:Conn_01x04_Pin
- added J22: USB_C_Receptacle_USB2.0_16P, Connector_USB:USB_C_Receptacle_G-Switch_GT-USB-7051x, symbol Connector:USB_C_Receptacle_USB2.0_16P
- added R69, R73: 5.1k, Resistor_SMD:R_0603_1608Metric, symbol Device:R_Small
Connections:
- net DN: now also J22.A7 (D-), J22.B7 (D-)
- net DP: now also J22.A6 (D+), J22.B6 (D+)
- net GND: now also J22.A1 (GND), J22.A12 (GND), J22.B1 (GND), J22.B12 (GND), J22.S1 (SHIELD), R69.2, R73.2
- net VBUS: now also J22.A4 (VBUS), J22.A9 (VBUS), J22.B4 (VBUS), J22.B9 (VBUS)
- new net: J22.B5 (CC2), R69.1
- new net: J22.A5 (CC1), R73.1
- no-connect marks 1 -> 3

Commit message: get ready for production fixes #24 fixes #25
Parts:
- J22: LCSC (none) -> C2843970
- R69, R73: LCSC C14675 -> C23186
Changed lines of the file:
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@@
 			)
 		)
-		(property "LCSC" "C14675"
+		(property "LCSC" "C23186"
 			(at 80.01 58.42 0)
 			(effects
@@
 			)
 		)
+		(property "LCSC" "C2843970"
+			(at 48.26 38.1 0)
+			(effects
+				(font
+					(size 1.27 1.27)
+				)
+				(hide yes)
+			)
+		)
 		(pin "B9"
 		)
@@
 			)
 		)
-		(property "LCSC" "C14675"
+		(property "LCSC" "C23186"
 			(at 88.9 58.42 0)
 			(effects
